File: MRCS-Integrated-Turnout-Controller.brd (EAGLE design)
At the start: 44.5 x 49.5 mm, 24 parts, among them U1 TC4428A, U2 Tiny85, U3 U3

Commit message: Changes to correct U1/U2 reversal on board labels
silk changes
Parts:
- C4, E$3: device SparkFun-Capacitors:CAP-PTH-SMALL -> SparkFun-Passives:CAP-PTH-SMALL
- J1: device con-molex:MRCS-156-LOCK -> SPCoast:KK-156-8-F
- moved J1 17.3 mm to (22.2, 41.3)
Routing:
- net S$20: track 10.2 -> 8.02 mm
- net S$11: track 9.53 -> 7.50 mm
Other:
- board text added: "00119-2021 v1.3a"
- board text added: "ACTPOS"
- board text added: "RN1"
- board text added: "T5"
- board text added: "T6"
- board text added: "U3"
- board text removed: "1130-2017 v1.3"
